File: Clock Board.kicad_pcb (KiCad board)
At the start: 2 copper layers, 80 x 50 mm, 29 parts, among them J2 Clk Output, J3 Clk Output, SW1 Single Step, SW2 Clk Select, U1 NE555P, U2 NE555P, U3 NE555P, U4 74HCT02, U6 74LS08

Commit message: PCBWay - Initial Design Submitted
Parts:
- added Ref1: MountingHole_2.2mm_M2, MountingHole:MountingHole_2.2mm_M2, F.Cu at (119.0, 62.0)
- added Ref2: MountingHole_2.2mm_M2, MountingHole:MountingHole_2.2mm_M2, F.Cu at (119.0, 106.0)
- added Ref3: MountingHole_2.2mm_M2, MountingHole:MountingHole_2.2mm_M2, F.Cu at (45.0, 106.0)
- added Ref4: MountingHole_2.2mm_M2, MountingHole:MountingHole_2.2mm_M2, F.Cu at (45.0, 62.0)
- D1: value LED -> Clk Out
- moved D1 2.96 mm to (116.3, 97.4)
- moved R7 2.83 mm to (109.3, 101.5)
- moved SW1 1.88 mm to (50.8, 101.7)
Routing:
- net Net-(U2-TRIG): track 58.8 -> 56.9 mm
- net Net-(J2-Pin_3): track 62.3 -> 60.6 mm
Other:
- board text added: "WayWayWay"

Commit message: Reverse diodes, increase text size on some labels
Parts:
- D1: value Clk Out -> LED
- moved D3 2.62 mm to (66.7, 95.6), turned to 180 degrees
- moved D2 2.54 mm to (76.2, 95.8), turned to 180 degrees
Connections:
- D2 pad 1: Net-(U1-OUT) -> Net-(D2-Pad1)
- D2 pad 2: Net-(D2-Pad2) -> Net-(U1-OUT)
- D3 pad 1: Net-(U2-OUT) -> Net-(D3-Pad1)
- D3 pad 2: Net-(D3-Pad2) -> Net-(U2-OUT)
- R8 pad 1: Net-(D2-Pad2) -> Net-(D2-Pad1)
- R9 pad 2: Net-(D3-Pad2) -> Net-(D3-Pad1)
Routing:
- net Net-(D2-Pad2): track 17.5 -> 0.00 mm
- net Net-(D2-Pad1): track 0.00 -> 17.5 mm
- net Net-(D3-Pad1): track 0.00 -> 13.2 mm
- net Net-(D3-Pad2): track 13.2 -> 0.00 mm
Other:
- board text added: "Tom Gambill v101"
- board text removed: "Tom Gambill v100"
